File: raspberry_pi_hat.kicad_pcb (KiCad board)
At the start: 2 copper layers, 65 x 56 mm, 34 parts, among them J1 CONN_JTAG, J3 Conn_01x08, J4 475890001, P1 CONN_02X20, U2 FT232H, Y1 CSTNE12M0G550000R0

Commit message: progress
Parts:
- renumbered J3 to ILI9341, J1 to JTAG
Other:
- board text added: "3V3"
- board text added: "BL"
- board text added: "CLK"
- board text added: "CORP"
- board text added: "DC"
- board text added: "DISPLAY"
- board text added: "GND"
- board text added: "GPIO06"
- board text added: "GPIO09"
- board text added: "GPIO10"
- board text added: "GPIO11"
- board text added: "GPIO13"
- board text added: "GPIO19"
- board text added: "MISO"
- board text added: "MOSI"
- board text added: "RST"
- board text added: "Raspberry Pi"
- board text added: "TCK"
- board text added: "TDI"
- board text added: "TDO"
- board text added: "TMS"
- board text added: "TRST"
- board text added: "ZOMBIE"
- board text added: "dev hat"

Commit message: progress
Parts:
- removed ILI9341: Conn_01x08, Connector_PinHeader_2.54mm:PinHeader_1x08_P2.54mm_Horizontal
- removed JTAG: CONN_JTAG, Connector_PinSocket_2.54mm:PinSocket_1x06_P2.54mm_Horizontal
- removed eeprom: 93LC56BT-I_OT, footprints:SOT95P280X145-6N
- added C12: 27pF, Capacitor_SMD:C_0201_0603Metric_Pad0.64x0.40mm_HandSolder, F.Cu at (228.8, 119.6)
- added C13: 27pF, Capacitor_SMD:C_0201_0603Metric_Pad0.64x0.40mm_HandSolder, F.Cu at (233.9, 119.5)
- added C14: 4.7uF, footprints:CAPPM2014X120N, F.Cu at (220.9, 120.4)
- added C15: 0.1uF, Capacitor_SMD:C_0201_0603Metric_Pad0.64x0.40mm_HandSolder, F.Cu at (232.2, 112.8)
- added C16: 0.1uF, Capacitor_SMD:C_0201_0603Metric_Pad0.64x0.40mm_HandSolder, F.Cu at (219.2, 115.4)
- added C17: 0.1uF, Capacitor_SMD:C_0201_0603Metric_Pad0.64x0.40mm_HandSolder, F.Cu at (224.6, 126.5)
- added J1: CONN_JTAG, Connector_PinSocket_2.54mm:PinSocket_1x06_P2.54mm_Horizontal, F.Cu at (210.2, 104.6)
- added J3: Conn_01x08, Connector_PinHeader_2.54mm:PinHeader_1x08_P2.54mm_Horizontal, F.Cu at (226.4, 138.5)
- added L4: 600R/0.5A, footprints:BLM21AG102BH1J, F.Cu at (236.8, 111.4)
- added R10: 10K, Resistor_SMD:R_0201_0603Metric_Pad0.64x0.40mm_HandSolder, F.Cu at (226.6, 127.1)
- added R6: 10K, Resistor_SMD:R_0201_0603Metric_Pad0.64x0.40mm_HandSolder, F.Cu at (224.8, 124.2)
- added R7: 39K, Resistor_SMD:R_0201_0603Metric_Pad0.64x0.40mm_HandSolder, F.Cu at (219.4, 113.3)
- added R8: 10K, Resistor_SMD:R_0201_0603Metric_Pad0.64x0.40mm_HandSolder, F.Cu at (220.0, 115.4)
- added R9: 10K, Resistor_SMD:R_0201_0603Metric_Pad0.64x0.40mm_HandSolder, F.Cu at (224.8, 125.2)
- added U1: 93LC56BT-I_OT, footprints:SOT95P280X145-6N, F.Cu at (227.9, 125.2)
- C1, C10, C11, C2, C4, C6, C9: footprint Capacitor_SMD:C_0504_1310Metric_Pad0.83x1.28mm_HandSolder -> Capacitor_SMD:C_0201_0603Metric_Pad0.64x0.40mm_HandSolder
- C3, C5, C7: footprint Capacitor_SMD:C_0504_1310Metric_Pad0.83x1.28mm_HandSolder -> footprints:CAPPM2014X120N
- C8: value 4.7uF -> 0.1uF; footprint Capacitor_SMD:C_0504_1310Metric_Pad0.83x1.28mm_HandSolder -> Capacitor_SMD:C_0201_0603Metric_Pad0.64x0.40mm_HandSolder
- D2: value PGB1010603NR -> PGB1010603NR (x2)
- J4: footprint footprints:CON00363_5_MOL_FIXED -> footprints:usb_mini
- L1, L2: value L -> 600R/0.5A; footprint Inductor_SMD:L_1008_2520Metric -> footprints:BLM21AG102BH1J
- R1: value R -> 220; footprint Resistor_SMD:R_0603_1608Metric -> Resistor_SMD:R_0201_0603Metric_Pad0.64x0.40mm_HandSolder
- R2: value 12K -> 12K / %1; footprint Resistor_SMD:R_0402_1005Metric_Pad0.72x0.64mm_HandSolder -> Resistor_SMD:R_0201_0603Metric_Pad0.64x0.40mm_HandSolder
- R3: value 2k2 -> 2K2; footprint Resistor_SMD:R_0402_1005Metric_Pad0.72x0.64mm_HandSolder -> Resistor_SMD:R_0201_0603Metric_Pad0.64x0.40mm_HandSolder
- R4, R5: footprint Resistor_SMD:R_0603_1608Metric -> Resistor_SMD:R_0201_0603Metric_Pad0.64x0.40mm_HandSolder
- moved C2 23.7 mm to (223.3, 119.3), turned to 90 degrees
- moved C1 23.3 mm to (222.6, 119.3), turned to 90 degrees
- moved R3 22.0 mm to (231.6, 125.3), turned to 90 degrees
- moved D4 21.9 mm to (226.5, 103.6), turned to -90 degrees
- moved C11 21.8 mm to (223.0, 106.9), turned to 90 degrees
- moved D5 20.6 mm to (228.2, 103.6), turned to -90 degrees
- moved R4 16.1 mm to (227.0, 106.8), turned to -90 degrees
- moved R5 15.0 mm to (227.8, 106.8), turned to -90 degrees
- moved C7 15.0 mm to (233.6, 112.0), turned to 90 degrees
- moved L1 12.9 mm to (236.8, 114.8), turned to 180 degrees
- moved C10 11.8 mm to (231.4, 110.9), turned to -90 degrees
- moved L2 11.7 mm to (214.4, 122.5)
- moved Y1 11.5 mm to (231.6, 119.8), turned to 0 degrees
- moved U2 10.8 mm to (225.7, 113.1), turned to 180 degrees
- moved C3 10.7 mm to (233.5, 116.1)
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Connections:
- net Net-(U2-REF) renamed /REF
- C1 pad 1: unconnected-(C1-Pad1) -> /GND
- C1 pad 2: /GND -> /VCCA
- C10 pad 1: /VCCIO -> +3V3
- C11 pad 1: /VCCIO -> +3V3
- C2 pad 1: unconnected-(C2-Pad1) -> /GND
- C2 pad 2: /GND -> /VCORE
- C5 pad 1: /VPLL -> /RPI_5V
- C6 pad 1: /VPLL -> /RPI_5V
- C7 pad 1: /vcc3v3 -> /VPLL
- C8 pad 1: /vcc3v3 -> +3V3
- C9 pad 1: /VCCIO -> +3V3
- D2 pad 2: /DM -> /DP
- D3 pad 2: /DP -> /DM
- J4 pad 1: /USB_5V -> Net-(J4-Pad1)
- L1 pad 1: /vcc3v3 -> +3V3
- L2 pad 1: /vcc3v3 -> Net-(J4-Pad1)
- L2 pad 2: /VPLL -> /VBUS
- U2 pad 12: /VCCIO -> +3V3
- U2 pad 24: /VCCIO -> +3V3
- U2 pad 31: unconnected-(U2-ACBUS7-Pad31) -> /AC7
- U2 pad 34: /VCCIO -> /#RESET
- U2 pad 37: unconnected-(C1-Pad1) -> /VCCA
- U2 pad 38: unconnected-(C2-Pad1) -> /VCORE
- U2 pad 39: /vcc3v3 -> +3V3
- U2 pad 40: /USB_5V -> /RPI_5V
- U2 pad 46: /VCCIO -> +3V3
Routing:
- net /GND: track 116.0 -> 40.9 mm, vias 3 -> 30
- net +3V3: track 0.00 -> 68.1 mm, vias 0 -> 8
- net /USB_5V: track 41.8 -> 0.00 mm, vias 2 -> 0
- net /RPI_5V: track 0.00 -> 41.2 mm, vias 0 -> 1
- net /vcc3v3: track 40.7 -> 0.00 mm, vias 4 -> 0
- net /RPI_3V3: track 55.4 -> 79.2 mm, vias 1 -> 4
- net /UART_RX: track 33.5 -> 18.3 mm
- net /VBUS: track 0.00 -> 11.4 mm
- net /DM: track 42.9 -> 31.7 mm
- net /UART_TX: track 33.7 -> 22.6 mm, vias 1 -> 3
- net Net-(J4-Pad1): track 0.00 -> 9.00 mm, vias 0 -> 2
- net /REF: track 2.84 -> 9.99 mm, vias 0 -> 2
- net /VCCIO: track 7.02 -> 0.00 mm
- net /DP: track 39.4 -> 32.9 mm, vias 0 -> 2
- net /DISPL_CLK: track 63.5 -> 57.0 mm
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- added copper zone on B.Cu, net /GND
Other:
- board text removed: "GPIO09"
- board text removed: "GPIO10"
- board text removed: "GPIO11"
- board text removed: "Raspberry Pi"
- board text removed: "dev hat"
